File: HBridgeMotorControl/HBridgeMotorControl.kicad_sch (KiCad schematic)
At the start: 13 parts, among them M1 Motor_DC, Q1 PNP, Q2 PNP, Q3 NPN, Q4 NPN

Commit message: add footprints
Parts:
- added BT1: Battery, Connector_PinHeader_2.54mm:PinHeader_1x02_P2.54mm_Vertical, symbol Device:Battery
- added J1: Conn_01x04, Connector_PinHeader_2.54mm:PinHeader_1x04_P2.54mm_Vertical, symbol Connector_Generic:Conn_01x04
- M1: footprint (none) -> Connector_PinHeader_2.54mm:PinHeader_1x02_P2.54mm_Vertical
- Q1, Q2, Q3, Q4: footprint (none) -> Package_TO_SOT_THT:TO-92_Inline
- R1, R2, R3, R4: footprint (none) -> Resistor_THT:R_Axial_DIN0207_L6.3mm_D2.5mm_P10.16mm_Horizontal
Connections:
- net GND: now reaches D3.2 (A), D4.2 (A), Q3.3 (E), Q4.3 (E)
- net GND: now also BT1.2 (-)
- net at D1.1 (K), D2.1 (K), Q1.3 (E)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: now also BT1.1 (+)
- net at R2.1: now also J1.2 (Pin_2)
- net at R4.2: now also J1.4 (Pin_4)
- net at R1.1: now also J1.1 (Pin_1)
- net at R3.2: now also J1.3 (Pin_3)
